Commit message: Added hand calibration

File: display/urdf/hand.urdf.xacro (robot description, xacro)
@@ -5,5 +5,5 @@
       <visual>
         <geometry>
-         <mesh filename="file://$(find display)/mesh/hand/hand.stl" scale="0.1 0.1 0.1"/>
+         <mesh filename="file://$(find display)/mesh/hand/total_hand.stl" scale="0.01 0.01 0.01"/>
         </geometry>
         <material name="${color}" />
